Commit message: moveJ using AR4 default

File: ar3_description/urdf/ar3.urdf (robot description, URDF)
Before this commit: robot ar3, 7 links, 6 joints
Joints:
- joint joint_1: axis 0 0 1 -> 0 0 -1
- joint joint_3: origin xyz=0.1525 -0.26414 0 rpy=3.3431E-16 -1.4164E-16 -1.4953816339 -> xyz=0.1525 -0.26414 0 rpy=0 0 -2.61799387799

File: ar3_description/urdf/ar3.urdf.xacro (robot description, xacro)
@@ -53,5 +53,5 @@
     <parent link="base_link"/>
     <child link="link_1"/>
-    <axis xyz="0 0 1"/>
+    <axis xyz="0 0 -1"/>
     <limit lower="-2.96706" upper="2.96706" effort="0" velocity="0"/>
   </joint>
@@ -108,5 +108,6 @@
   </link>
   <joint name="joint_3" type="revolute">
-    <origin rpy="0 0 -1.04720367321" xyz="0.1525 -0.26414 0"/>
+    <!-- <origin rpy="0 0 -1.04720367321" xyz="0.1525 -0.26414 0"/> -->
+    <origin rpy="0 0 -2.61799387799" xyz="0.1525 -0.26414 0"/>
     <parent link="link_2"/>
     <child link="link_3"/>

File: ar3_description/urdf/ar3_gazebo.urdf.xacro (robot description, xacro)
@@ -114,9 +114,9 @@
   </link>
   <joint name="joint_3" type="revolute">
-    <origin rpy="0 0 -1.04720367321" xyz="0.1525 -0.26414 0"/>
+    <origin rpy="0 0 -2.61799387799" xyz="0.1525 -0.26414 0"/>
     <parent link="link_2"/>
     <child link="link_3"/>
     <axis xyz="0 0 -1"/>
-    <limit lower="0.0174533" upper="2.5080381" effort="100" velocity="100"/>
+    <limit lower="-1.55334 " upper="20.907571" effort="100" velocity="100"/>
   </joint>
   <link name="link_4">
